Commit message: feat: 按实测舵机参数更新URDF，加入浏览器3D预览和真实夹爪STL
- 舵机型号: DS3218MG -> WHEELTEC S20F (180deg x2 + 270deg x3) + 360deg速度舵机
- wrist_roll 改为 continuous joint (速度舵机无位置反馈)
- 夹爪改为单舵机驱动 + finger_right mimic
- 关节限位按实测脉宽范围重新计算
- 新增 k3b_arm_preview.html 浏览器3D预览
- 夹爪使用商家提供的真实STL模型(新款机械爪)
- 更新所有文档的舵机编号与关节映射表

File: k3b_arm_urdf/k3b_arm.urdf (robot description, URDF)
Before this commit: robot k3b_arm, 11 links, 10 joints
Joints:
- joint elbow_pitch: limit lower=-1.5708 upper=1.5708 effort=12.0 velocity=1.5 -> lower=-2.356 upper=2.356 effort=12.0 velocity=1.5
- joint finger_left_joint: limit lower=0 upper=0.5 effort=3.0 velocity=2.0 -> lower=0 upper=1.022 effort=3.0 velocity=2.0
- joint finger_right_joint: limit lower=0 upper=0.5 effort=3.0 velocity=2.0 -> lower=0 upper=1.022 effort=3.0 velocity=2.0; mimic (none) -> joint=finger_left_joint multiplier=-1.0 offset=0
- joint shoulder_pitch: limit lower=-1.5708 upper=1.5708 effort=15.0 velocity=1.5 -> lower=-1.763 upper=1.763 effort=15.0 velocity=1.5
- joint wrist_pitch: limit lower=-1.5708 upper=1.5708 effort=8.0 velocity=1.5 -> lower=-2.234 upper=2.234 effort=8.0 velocity=1.5
- joint wrist_roll: limit lower=-1.5708 upper=1.5708 effort=8.0 velocity=1.5 -> effort=5.0 velocity=2; type revolute -> continuous

File: k3b_arm_urdf/k3b_arm.urdf.xacro (robot description, xacro)
@@ -1,38 +1,52 @@
 <?xml version="1.0"?>
 <!--
-  K3B 六轴机械臂 URDF (xacro 参数化版)
-  依据：淘宝在售 6 自由度舵机机械臂 DIY 套件实物图
-  结构：base_yaw(J1) -> shoulder_pitch(J2) -> elbow_pitch(J3)
-        -> wrist_pitch(J4) -> wrist_roll(J5) -> 两指夹爪(J6)
-  执行器：DS3218MG 标准 PWM 舵机（500-2500us，中点1500us，默认180°）
-  说明：杆长为按图片标注的估算值，实机前必须按实物实测校准：
-        1) 实测各关节轴到轴的直线距离（杆长）
-        2) 实测每个舵机的关节角限位（机械限位，避免卡死）
-        3) 确认各关节旋转轴朝向（本模型按常见正装结构取 Y/Z 轴）
+  K3B 机械臂 URDF (xacro 参数化版) — 按实测舵机参数修订
+  硬件：WHEELTEC S20F 数字舵机 ×5 + 360° 速度舵机 ×1
+  结构链：
+    base_yaw(J1,S2,180deg) -> shoulder_pitch(J2,S3,270deg)
+    -> elbow_pitch(J3,S4,270deg) -> wrist_pitch(J4,S5,270deg)
+    -> wrist_roll(360deg速度舵机, continuous) -> gripper
+    -> finger(S1,180deg, 夹爪开合)
+  舵机->关节映射（实测 2026-10-25）：
+    S1 850~1500us  上电850us  = 夹爪开合(OPEN=850/CLOSE=1500)
+    S2 500~2500us  上电1500us = base_yaw
+    S3 500~2000us  上电2000us = shoulder_pitch
+    S4 500~2500us  上电500us  = elbow_pitch
+    S5 600~2500us  上电1500us = wrist_pitch
+    360度速度舵机             = wrist_roll（控速度，不控位置）
+  角度换算：
+    180deg 舵机: angle_deg = (pulse_us - 500) * 180 / 2000
+    270deg 舵机: angle_deg = (pulse_us - 500) * 270 / 2000
+  零点策略：joint=0 对应机械臂直立位（臂伸直向上），
+            限位围绕直立位对称设置；实物校准后微调下方 limit_* 参数。
   用法：xacro k3b_arm.urdf.xacro > k3b_arm.urdf
 -->
 <robot name="k3b_arm" xmlns:xacro="http://www.ros.org/wiki/xacro">
-  <!-- ============ 参数（按图估算，需实测校准） ============ -->
+  <!-- ============ 几何参数（杆长需实测替换） ============ -->
   <xacro:property name="pi" value="3.141592653589793"/>
-  <xacro:property name="base_height"    value="0.14"/>   <!-- 底座高度(估算) -->
-  <xacro:property name="base_radius"    value="0.05"/>   <!-- 底座半径(估算) -->
-  <xacro:property name="upper_arm_len"  value="0.43"/>   <!-- 大臂长度，图中 43cm -->
-  <xacro:property name="forearm_len"    value="0.313"/>  <!-- 前臂长度，图中 31.3cm -->
-  <xacro:property name="wrist_len"      value="0.09"/>   <!-- 腕部长度，图中 9cm -->
-  <xacro:property name="gripper_len"    value="0.10"/>   <!-- 夹爪长度(估算) -->
-  <xacro:property name="joint_speed"    value="1.5"/>    <!-- 舵机额定速度 rad/s(估算) -->
-  <!-- 默认关节限位：按 DS3218MG 舵机默认 180° 量程设为 ±90°；
-       实际机械限位(支架阻挡)以实测为准，若舵机为 270° 版可放宽 -->
-  <xacro:property name="lim_base"   value="1.5708"/>  <!-- ±90° -->
-  <xacro:property name="lim_should" value="1.5708"/>  <!-- ±90° -->
-  <xacro:property name="lim_elbow"  value="1.5708"/>  <!-- ±90° -->
-  <xacro:property name="lim_wpitch" value="1.5708"/>  <!-- ±90° -->
-  <xacro:property name="lim_wroll"  value="1.5708"/>  <!-- ±90° -->
-  <xacro:property name="lim_finger" value="0.6"/>
+  <xacro:property name="base_height"    value="0.14"/>
+  <xacro:property name="base_radius"    value="0.05"/>
+  <xacro:property name="upper_arm_len"  value="0.43"/>   <!-- 实测替换 -->
+  <xacro:property name="forearm_len"    value="0.313"/>   <!-- 实测替换 -->
+  <xacro:property name="wrist_len"      value="0.09"/>    <!-- 实测替换 -->
+  <xacro:property name="gripper_len"    value="0.10"/>
+  <!-- ============ 关节限位（rad，按实测脉宽范围+中点=直立位换算） ============
+       S2 base_yaw    180deg, 500~2500us, 中点1500us=直立 -> ±90deg  -->
+  <xacro:property name="lim_base"      value="1.5708"/>   <!-- ±90deg -->
+  <!-- S3 shoulder_pitch 270deg, 500~2000us, 中点1250us=直立, 行程202.5deg -> ±101deg -->
+  <xacro:property name="lim_should"    value="1.763"/>    <!-- ±101deg，保守取整 -->
+  <!-- S4 elbow_pitch  270deg, 500~2500us, 中点1500us=直立, 行程270deg -> ±135deg -->
+  <xacro:property name="lim_elbow"      value="2.356"/>    <!-- ±135deg -->
+  <!-- S5 wrist_pitch  270deg, 600~2500us, 中点1550us=直立, 行程256.5deg -> ±128deg -->
+  <xacro:property name="lim_wpitch"     value="2.234"/>    <!-- ±128deg -->
+  <!-- S1 finger       180deg, 850~1500us, 行程58.5deg, 0=闭合/正=张开 -->
+  <xacro:property name="lim_finger"     value="1.022"/>    <!-- 58.5deg -->
+  <xacro:property name="joint_speed"   value="1.5"/>      <!-- rad/s 估算 -->
+  <xacro:property name="roll_speed"     value="2.0"/>      <!-- 360deg速度舵机 rad/s -->
   <!-- ============ 颜色 ============ -->
-  <material name="base_mat"> <color rgba="0.15 0.18 0.24 1.0"/> </material>
-  <material name="link_mat"> <color rgba="0.35 0.42 0.52 1.0"/> </material>
-  <material name="joint_mat"><color rgba="0.80 0.52 0.20 1.0"/> </material>
-  <material name="grip_mat"> <color rgba="0.20 0.65 0.55 1.0"/> </material>
+  <material name="base_mat">  <color rgba="0.15 0.18 0.24 1.0"/> </material>
+  <material name="link_mat">  <color rgba="0.35 0.42 0.52 1.0"/> </material>
+  <material name="joint_mat"> <color rgba="0.80 0.52 0.20 1.0"/> </material>
+  <material name="grip_mat">  <color rgba="0.20 0.65 0.55 1.0"/> </material>
   <!-- ============ 底座 ============ -->
   <link name="base_link">
@@ -51,5 +65,5 @@
     </inertial>
   </link>
-  <!-- ============ J1 底座偏航 ============ -->
+  <!-- ============ J1 base_yaw (S2, 180deg) ============ -->
   <link name="base_yaw_link">
     <visual>
@@ -75,5 +89,5 @@
     <dynamics damping="0.2" friction="0.1"/>
   </joint>
-  <!-- ============ J2 肩俯仰 ============ -->
+  <!-- ============ J2 shoulder_pitch (S3, 270deg) ============ -->
   <link name="upper_arm_link">
     <visual>
@@ -99,5 +113,5 @@
     <dynamics damping="0.2" friction="0.1"/>
   </joint>
-  <!-- ============ J3 肘俯仰 ============ -->
+  <!-- ============ J3 elbow_pitch (S4, 270deg) ============ -->
   <link name="forearm_link">
     <visual>
@@ -123,5 +137,5 @@
     <dynamics damping="0.2" friction="0.1"/>
   </joint>
-  <!-- ============ J4 腕俯仰 ============ -->
+  <!-- ============ J4 wrist_pitch (S5, 270deg) ============ -->
   <link name="wrist_link">
     <visual>
@@ -147,5 +161,8 @@
     <dynamics damping="0.15" friction="0.1"/>
   </joint>
-  <!-- ============ J5 腕滚转 ============ -->
+  <!-- ============ J5 wrist_roll (360deg 速度舵机, continuous) ============
+       速度舵机无位置反馈，控转速不控角度；URDF 用 continuous joint 表示。
+       注意：MoveIt 规划组里不要把它当位置关节做逆解，
+       它只在实机/仿真里做连续旋转速度控制。 -->
   <link name="wrist_roll_link">
     <visual>
@@ -163,11 +180,11 @@
     </inertial>
   </link>
-  <joint name="wrist_roll" type="revolute">
+  <joint name="wrist_roll" type="continuous">
     <parent link="wrist_link"/>
     <child link="wrist_roll_link"/>
     <origin xyz="0 0 ${wrist_len}" rpy="0 0 0"/>
     <axis xyz="0 0 1"/>
-    <limit lower="-${lim_wroll}" upper="${lim_wroll}" effort="8.0" velocity="${joint_speed}"/>
-    <dynamics damping="0.15" friction="0.1"/>
+    <limit effort="5.0" velocity="${roll_speed}"/>
+    <dynamics damping="0.1" friction="0.05"/>
   </joint>
   <!-- ============ 夹爪底座(固定) ============ -->
@@ -199,5 +216,8 @@
     <origin xyz="0 0 0.05" rpy="0 0 0"/>
   </joint>
-  <!-- ============ J6 左指 ============ -->
+  <!-- ============ 夹爪驱动指 (S1, 180deg, 850~1500us) ============
+       单舵机通过连杆驱动两指同步开合。
+       0 = 闭合(CLOSE=1500us)，正 = 张开(OPEN=850us)。
+       右指通过 mimic 跟随左指，方向反向。 -->
   <link name="finger_left_link">
     <visual>
@@ -222,5 +242,5 @@
     <limit lower="0" upper="${lim_finger}" effort="3.0" velocity="2.0"/>
   </joint>
-  <!-- ============ J6 右指 ============ -->
+  <!-- ============ 夹爪从动指（mimic 左指） ============ -->
   <link name="finger_right_link">
     <visual>
@@ -244,4 +264,5 @@
     <axis xyz="0 1 0"/>
     <limit lower="0" upper="${lim_finger}" effort="3.0" velocity="2.0"/>
+    <mimic joint="finger_left_joint" multiplier="-1.0" offset="0"/>
   </joint>
   <!-- 世界->底座，方便 RViz 固定 -->

Commit message: feat(gripper): 夹爪拆成壳体+左指+右指，改为 prismatic 可开合
之前夹爪只能看不能动：finger_left/right_link 里没有任何 <visual>，
整爪 part_claw.stl 被当成刚体挂在 gripper_base_link 上，
拖滑块时关节值在变、画面不动。

- tools/split_claw.py：按连通分量把 part_claw.stl（21 个零件的刚性
  装配体）拆成 claw_body / finger_left / finger_right 三个 STL。
  判据：长薄板（sizeZ>56mm, sizeX<20mm, sizeY<6mm）为指片，
  按质心 X 与对称面 X=2.75mm 分左右，其余归壳体。
- xacro：finger_left/right_joint 由 revolute(Y) 改为 prismatic(X)，
  与「S1 转舵盘 → 四连杆 → 指片直线开合」的实际运动一致；
  lim_finger(1.021 rad) 换成 finger_stroke(0.010 m)。
  实测指间缝 7.5mm（合拢）→ 27.5mm（全开），两指仍由 mimic -1 联动。
- preview.html：applyAll 支持 prismatic（沿 axis 平移，不改姿态），
  滑块副值与读数按关节类型切换（mm / °），复位改为重建面板。
- tools/shot.js：CDP 截图 + 页面内注入 JS 自检，替掉在新版 Edge 上
  不出文件的 --headless --screenshot。
- 文档同步：夹爪关节表、网格清单、机械爪拆分判据、待校准项。

验证：指间缝 7.5 → 17.5 → 27.5 mm 随滑块线性变化（三档实测）。

File: k3b_arm_urdf/k3b_arm.urdf (robot description, URDF)
Before this commit: robot k3b_arm, 11 links, 10 joints
Links:
- link finger_left_link: mass 0.02 -> 0.03; geometry collision box size=0.0169 0.005 0.0593; visual mesh filename=package://k3b_arm_urdf/meshes/finger_left.stl
- link finger_right_link: mass 0.02 -> 0.03; geometry collision box size=0.0169 0.005 0.0593; visual mesh filename=package://k3b_arm_urdf/meshes/finger_right.stl
- link gripper_base_link: geometry collision box size=0.032 0.026 0.016; collision box size=0.060 0.022 0.078
Joints:
- joint finger_left_joint: axis 0 1 0 -> 1 0 0; limit lower=0 upper=1.021 effort=3.0 velocity=2.0 -> lower=0 upper=0.01 effort=12.0 velocity=0.04; origin xyz=0 0.018 0.040 rpy=0 0 0 -> xyz=0 0 0 rpy=0 0 0; type revolute -> prismatic
- joint finger_right_joint: axis 0 1 0 -> 1 0 0; limit lower=-1.021 upper=0 effort=3.0 velocity=2.0 -> lower=-0.01 upper=0 effort=12.0 velocity=0.04; origin xyz=0 -0.018 0.040 rpy=0 0 0 -> xyz=0 0 0 rpy=0 0 0; type revolute -> prismatic

File: k3b_arm_urdf/k3b_arm.urdf.xacro (robot description, xacro)
@@ -4,5 +4,5 @@
   =============================================================
   执行器实测映射（2026-10-25）
-  S1  180° 位置   脉宽 850~1500   上电 850    → finger_left      限位 0~58.5°
+  S1  180° 位置   脉宽 850~1500   上电 850    → finger_left      行程 0~10mm
   S2  180° 位置   脉宽 500~2500   上电 1500   → base_yaw         限位 ±90°
   S3  270° 位置   脉宽 500~2000   上电 2000   → shoulder_pitch   限位 ±101°
@@ -37,6 +37,7 @@
   <xacro:property name="lim_elbow"  value="2.3562"/>   <!-- S4  270°  ±135° -->
   <xacro:property name="lim_wpitch" value="2.2340"/>   <!-- S5  270°  ±128° -->
-  <xacro:property name="lim_finger" value="1.0210"/>   <!-- S1  180°  0~58.5° -->
   <xacro:property name="joint_speed" value="1.5"/>
+  <!-- 夹爪：单指行程（m）。0 = 合拢（指间缝 7.5mm），0.010 = 张开（缝 27.5mm） -->
+  <xacro:property name="finger_stroke" value="0.010"/>
   <!-- ================= 网格 ================= -->
   <xacro:property name="mesh_dir" value="package://k3b_arm_urdf/meshes/"/>
@@ -285,7 +286,7 @@
       <material name="servo_mat"/>
     </visual>
-    <!-- 新款机械爪（铝制平行连杆）：整机刚性挂载 -->
-    <visual>
-      <geometry><mesh filename="${mesh_dir}part_claw.stl"/></geometry>
+    <!-- 新款机械爪（铝制平行连杆）：壳体 / 连杆部分 -->
+    <visual>
+      <geometry><mesh filename="${mesh_dir}claw_body.stl"/></geometry>
       <origin xyz="0 0 0.040" rpy="0 ${pi} 0"/>
       <material name="metal_mat"/>
@@ -294,4 +295,8 @@
       <geometry><box size="0.032 0.026 0.016"/></geometry>
       <origin xyz="0 0 0.014" rpy="0 0 0"/>
+    </collision>
+    <collision>
+      <geometry><box size="0.060 0.022 0.078"/></geometry>
+      <origin xyz="0 0 0.025" rpy="0 0 0"/>
     </collision>
     <inertial>
@@ -313,31 +318,56 @@
   </joint>
   <!-- ================= J6 左指（S1 驱动） ================= -->
-  <!-- 视觉由机械爪整机承担，这里只保留运动学链供 MoveIt 使用 -->
+  <!-- 平行连杆爪的等效自由度：指片沿 +X 平移（不是绕轴摆动）。
+       实机是 S1 转舵盘 → 四连杆 → 指片直线开合，中间连杆的转角对外不可见，
+       URDF 里直接把它折成 prismatic，MoveIt 侧也更好规划。
+       指片网格保留整爪坐标系，靠 visual/origin 对齐，两指在 0 位严丝合缝。 -->
   <link name="finger_left_link">
-    <inertial>
-      <mass value="0.02"/>
-      <inertia ixx="0.00001" ixy="0.0" ixz="0.0" iyy="0.00001" iyz="0.0" izz="0.00001"/>
-    </inertial>
-  </link>
-  <joint name="finger_left_joint" type="revolute">
+    <visual>
+      <geometry><mesh filename="${mesh_dir}finger_left.stl"/></geometry>
+      <origin xyz="0 0 0.040" rpy="0 ${pi} 0"/>
+      <material name="link_mat"/>
+    </visual>
+    <!-- 指片实测 X 1.0~17.9  Y -4.0~1.0  Z 35.0~94.3 (mm) -->
+    <collision>
+      <geometry><box size="0.0169 0.005 0.0593"/></geometry>
+      <origin xyz="0.00945 -0.0015 0.06465" rpy="0 0 0"/>
+    </collision>
+    <inertial>
+      <mass value="0.03"/>
+      <inertia ixx="0.00002" ixy="0.0" ixz="0.0" iyy="0.00002" iyz="0.0" izz="0.00001"/>
+    </inertial>
+  </link>
+  <joint name="finger_left_joint" type="prismatic">
     <parent link="gripper_base_link"/>
     <child link="finger_left_link"/>
-    <origin xyz="0 0.018 0.040" rpy="0 0 0"/>
-    <axis xyz="0 1 0"/>
-    <limit lower="0" upper="${lim_finger}" effort="3.0" velocity="2.0"/>
+    <origin xyz="0 0 0" rpy="0 0 0"/>
+    <axis xyz="1 0 0"/>
+    <limit lower="0" upper="${finger_stroke}" effort="12.0" velocity="0.04"/>
+    <dynamics damping="2.0" friction="0.5"/>
   </joint>
   <!-- ================= J6 右指（mimic 跟随左指） ================= -->
   <link name="finger_right_link">
-    <inertial>
-      <mass value="0.02"/>
-      <inertia ixx="0.00001" ixy="0.0" ixz="0.0" iyy="0.00001" iyz="0.0" izz="0.00001"/>
-    </inertial>
-  </link>
-  <joint name="finger_right_joint" type="revolute">
+    <visual>
+      <geometry><mesh filename="${mesh_dir}finger_right.stl"/></geometry>
+      <origin xyz="0 0 0.040" rpy="0 ${pi} 0"/>
+      <material name="link_mat"/>
+    </visual>
+    <!-- 指片实测 X -23.4~-6.5  Y -4.0~1.0  Z 35.0~94.3 (mm) -->
+    <collision>
+      <geometry><box size="0.0169 0.005 0.0593"/></geometry>
+      <origin xyz="-0.01495 -0.0015 0.06465" rpy="0 0 0"/>
+    </collision>
+    <inertial>
+      <mass value="0.03"/>
+      <inertia ixx="0.00002" ixy="0.0" ixz="0.0" iyy="0.00002" iyz="0.0" izz="0.00001"/>
+    </inertial>
+  </link>
+  <joint name="finger_right_joint" type="prismatic">
     <parent link="gripper_base_link"/>
     <child link="finger_right_link"/>
-    <origin xyz="0 -0.018 0.040" rpy="0 0 0"/>
-    <axis xyz="0 1 0"/>
-    <limit lower="-${lim_finger}" upper="0" effort="3.0" velocity="2.0"/>
+    <origin xyz="0 0 0" rpy="0 0 0"/>
+    <axis xyz="1 0 0"/>
+    <limit lower="-${finger_stroke}" upper="0" effort="12.0" velocity="0.04"/>
+    <dynamics damping="2.0" friction="0.5"/>
     <mimic joint="finger_left_joint" multiplier="-1" offset="0"/>
   </joint>
