Commit message: feat(gripper): 按实测定重定位夹爪，指片改回齿轮驱动的转动关节
用户补充了机构与尺寸：S1 输出轴带一只齿轮，与指片根部齿轮啮合，
逆时针张开、顺时针闭合；齿轮中心→爪尖 85mm（合拢）/ 70mm（全开）、
腕滚转输出→爪尖 110mm、全开两爪尖内距 55mm。

三条实测立刻定死了几何：
- 爪长 108.6mm 而「腕滚转→爪尖」只有 110mm，说明爪顶几乎贴在腕轴上；
  之前 claw 挂在 0.040 处，导致腕→爪尖 122mm、整机偏高 12mm。
  claw_z 改 0.0277 → 腕→爪尖 110.0mm，整机高度 55.7 → 54.5cm。
- 「齿轮中心→爪尖 85mm」反推齿轮在 claw Z=+30.7（= 爪顶下 23.6mm），
  正好落在爪体上那 4 个 6mm 凸台的高度，S1 因此从原来的
  (0.010,-0.012,0.008) 移到 (-0.00275,0.013,-0.003)，
  机身贴爪体 +Y 面外挂 —— 与实拍一致（不是之前的"悬空外挂 5cm"）。

指片运动由 prismatic 改回 revolute：
- 实测「全开时爪尖离齿轮 70mm < 合拢 85mm」只有转动能做出来，
  平移关节做不到，照片里张开也是明显的 V 字。
- 转轴取指片自身顶端中心；tools/solve_gripper.py 按合拢/全开两态反解，
  左右两指算出的转角比 = -1.000，与一对啮合齿轮的行为完全吻合，
  所以 finger_right 继续用 mimic -1（这次是有物理依据的，不是凑的）。
- lim_finger = 0.412rad(23.6°)，指间内距 7.5mm → 55.2mm（实测 55）。

preview.html：S1 标签注明「齿轮」，revolute/prismatic 两条分支都保留。
新增 tools/solve_gripper.py（实测值 → 装配基准 + 转角反解）。

验证（页面内量 mesh 顶点，强制 updateMatrixWorld）：
  合拢 内距 7.5mm / 齿轮→爪尖 85.1 / 腕→爪尖 110.0
  全开 内距 55.2mm / 齿轮→爪尖 87.8 / 腕→爪尖 108.4

遗留：全开时「齿轮→爪尖 70mm」与「内距 55mm」在现有爪形下无法同时成立
（模型给 87.8），已记入 README 待校准项，需要重新确认量的是哪个点。

File: k3b_arm_urdf/k3b_arm.urdf (robot description, URDF)
Before this commit: robot k3b_arm, 11 links, 10 joints
Links:
- link gripper_base_link: geometry collision box size=0.060 0.022 0.078; visual mesh filename=package://k3b_arm_urdf/meshes/claw_body.stl
Joints:
- joint finger_left_joint: axis 1 0 0 -> 0 1 0; limit lower=0 upper=0.01 effort=12.0 velocity=0.04 -> lower=0 upper=0.412 effort=12.0 velocity=1.5; origin xyz=0 0 0 rpy=0 0 0 -> xyz=0.00945 0 0.0227 rpy=0 0 0; type prismatic -> revolute
- joint finger_right_joint: axis 1 0 0 -> 0 1 0; limit lower=-0.01 upper=0 effort=12.0 velocity=0.04 -> lower=-0.412 upper=0 effort=12.0 velocity=1.5; origin xyz=0 0 0 rpy=0 0 0 -> xyz=-0.01495 0 0.0227 rpy=0 0 0; type prismatic -> revolute
- joint tool0_joint: origin xyz=0 0 0.096 rpy=0 0 0 -> xyz=0 0 0.082 rpy=0 0 0

File: k3b_arm_urdf/k3b_arm.urdf.xacro (robot description, xacro)
@@ -38,6 +38,22 @@
   <xacro:property name="lim_wpitch" value="2.2340"/>   <!-- S5  270°  ±128° -->
   <xacro:property name="joint_speed" value="1.5"/>
-  <!-- 夹爪：单指行程（m）。0 = 合拢（指间缝 7.5mm），0.010 = 张开（缝 27.5mm） -->
-  <xacro:property name="finger_stroke" value="0.010"/>
+  <!-- ===== 夹爪（实测定，见 tools/solve_gripper.py） =====
+       claw 网格自己的坐标系：爪尖 Z=-54.3、爪顶 Z=+54.3、厚 Y=+-11
+       齿轮中心 = 爪尖往 +Z 量 85mm  =>  claw Z=+30.7
+       腕滚转输出 -> 爪尖 110mm、爪长 108.6mm  =>  爪顶几乎贴住腕轴
+       claw 网格原点距 gripper_base = 54.3 - 28 + 1.4 = 27.7mm -->
+  <xacro:property name="claw_z" value="0.0277"/>
+  <xacro:property name="gear_x" value="-0.00275"/>   <!-- 齿轮中心，claw X=+2.75 镜像后 -->
+  <xacro:property name="gear_z" value="-0.0030"/>    <!-- 齿轮中心，爪顶下 23.6mm -->
+  <!-- 指片转角限位：0 = 合拢（内距 7.5mm），0.400rad(22.9°) = 全开（内距 55mm） -->
+  <xacro:property name="lim_finger" value="0.412"/>
+  <!-- 指片转轴（取指片顶端中心），claw 系 -> link 系后 -->
+  <xacro:property name="finger_piv_lx" value="0.00945"/>
+  <xacro:property name="finger_piv_rx" value="-0.01495"/>
+  <xacro:property name="finger_piv_z" value="0.0227"/>
+  <!-- 指片 visual 原点补偿：claw_z - 转轴 z（转轴在指片顶端，不在 claw 原点） -->
+  <xacro:property name="finger_vis_off" value="${claw_z - finger_piv_z}"/>
+  <xacro:property name="finger_half_w" value="0.00845"/>  <!-- 指片半宽（X） -->
+  <xacro:property name="finger_len" value="0.0593"/>      <!-- 指片长（Z） -->
   <!-- ================= 网格 ================= -->
   <xacro:property name="mesh_dir" value="package://k3b_arm_urdf/meshes/"/>
@@ -274,29 +290,23 @@
   </joint>
   <!-- ================= 夹爪 ================= -->
+  <!-- 装配基准由实测定（见 tools/solve_gripper.py）：
+       齿轮中心 -> 爪尖 85mm，腕滚转输出 -> 爪尖 110mm，爪长 108.6mm
+       所以爪顶几乎就贴在腕滚转轴上，claw 网格原点距 gripper_base 27.7mm。 -->
   <link name="gripper_base_link">
-    <visual>
-      <geometry><box size="0.032 0.026 0.016"/></geometry>
-      <origin xyz="0 0 0.014" rpy="0 0 0"/>
-      <material name="bracket_mat"/>
-    </visual>
-    <!-- S1：驱动夹爪开合，轴朝 +Y -->
-    <visual>
-      <geometry><mesh filename="${mesh_dir}s20f.stl"/></geometry>
-      <origin xyz="${s20f_xoff} -0.012 0.008" rpy="${servo_y_rpy}"/>
-      <material name="servo_mat"/>
-    </visual>
-    <!-- 新款机械爪（铝制平行连杆）：壳体 / 连杆部分 -->
+    <!-- S1：输出轴接一只齿轮（= 齿轮中心），机身从爪体 +Y 面外挂 -->
+    <visual>
+      <geometry><mesh filename="${mesh_dir}s20f.stl"/></geometry>
+      <origin xyz="${gear_x} 0.013 ${gear_z}" rpy="${pi/2} 0 0"/>
+      <material name="servo_mat"/>
+    </visual>
+    <!-- 新款机械爪：壳体 + 平行连杆 + 齿轮组 -->
     <visual>
       <geometry><mesh filename="${mesh_dir}claw_body.stl"/></geometry>
-      <origin xyz="0 0 0.040" rpy="0 ${pi} 0"/>
+      <origin xyz="0 0 ${claw_z}" rpy="0 ${pi} 0"/>
       <material name="metal_mat"/>
     </visual>
     <collision>
-      <geometry><box size="0.032 0.026 0.016"/></geometry>
-      <origin xyz="0 0 0.014" rpy="0 0 0"/>
-    </collision>
-    <collision>
       <geometry><box size="0.060 0.022 0.078"/></geometry>
-      <origin xyz="0 0 0.025" rpy="0 0 0"/>
+      <origin xyz="0 0 0.0124" rpy="0 0 0"/>
     </collision>
     <inertial>
@@ -310,26 +320,25 @@
     <origin xyz="0 0 0.028" rpy="0 0 0"/>
   </joint>
-  <!-- 末端工具坐标系（抓取参考点，落在爪尖附近） -->
+  <!-- 末端工具坐标系（抓取参考点，落在爪尖） -->
   <link name="tool0"/>
   <joint name="tool0_joint" type="fixed">
     <parent link="gripper_base_link"/>
     <child link="tool0"/>
-    <origin xyz="0 0 0.096" rpy="0 0 0"/>
-  </joint>
-  <!-- ================= J6 左指（S1 驱动） ================= -->
-  <!-- 平行连杆爪的等效自由度：指片沿 +X 平移（不是绕轴摆动）。
-       实机是 S1 转舵盘 → 四连杆 → 指片直线开合，中间连杆的转角对外不可见，
-       URDF 里直接把它折成 prismatic，MoveIt 侧也更好规划。
-       指片网格保留整爪坐标系，靠 visual/origin 对齐，两指在 0 位严丝合缝。 -->
+    <origin xyz="0 0 0.082" rpy="0 0 0"/>
+  </joint>
+  <!-- ================= J6 左指（S1 经齿轮驱动） ================= -->
+  <!-- 机构：S1 输出轴带一只齿轮，与指片根部的齿轮啮合；两齿轮转向相反，
+       所以两指反向等角摆开 —— 正好就是 mimic multiplier=-1。
+       指片绕自身顶端中心转动（取该点为转轴），0 = 合拢，0.400rad = 全开。 -->
   <link name="finger_left_link">
     <visual>
       <geometry><mesh filename="${mesh_dir}finger_left.stl"/></geometry>
-      <origin xyz="0 0 0.040" rpy="0 ${pi} 0"/>
+      <origin xyz="${-finger_piv_lx} 0 ${finger_vis_off}" rpy="0 ${pi} 0"/>
       <material name="link_mat"/>
     </visual>
-    <!-- 指片实测 X 1.0~17.9  Y -4.0~1.0  Z 35.0~94.3 (mm) -->
-    <collision>
-      <geometry><box size="0.0169 0.005 0.0593"/></geometry>
-      <origin xyz="0.00945 -0.0015 0.06465" rpy="0 0 0"/>
+    <!-- 转轴系下：X ±8.45、Y -4..1、Z 0..59.3 (mm) -->
+    <collision>
+      <geometry><box size="${finger_half_w*2} 0.005 ${finger_len}"/></geometry>
+      <origin xyz="0 -0.0015 ${finger_len/2}" rpy="0 0 0"/>
     </collision>
     <inertial>
@@ -338,23 +347,22 @@
     </inertial>
   </link>
-  <joint name="finger_left_joint" type="prismatic">
+  <joint name="finger_left_joint" type="revolute">
     <parent link="gripper_base_link"/>
     <child link="finger_left_link"/>
-    <origin xyz="0 0 0" rpy="0 0 0"/>
-    <axis xyz="1 0 0"/>
-    <limit lower="0" upper="${finger_stroke}" effort="12.0" velocity="0.04"/>
-    <dynamics damping="2.0" friction="0.5"/>
-  </joint>
-  <!-- ================= J6 右指（mimic 跟随左指） ================= -->
+    <origin xyz="${finger_piv_lx} 0 ${finger_piv_z}" rpy="0 0 0"/>
+    <axis xyz="0 1 0"/>
+    <limit lower="0" upper="${lim_finger}" effort="12.0" velocity="1.5"/>
+    <dynamics damping="2.0" friction="0.4"/>
+  </joint>
+  <!-- ================= J6 右指（齿轮啮合，反向跟随） ================= -->
   <link name="finger_right_link">
     <visual>
       <geometry><mesh filename="${mesh_dir}finger_right.stl"/></geometry>
-      <origin xyz="0 0 0.040" rpy="0 ${pi} 0"/>
+      <origin xyz="${-finger_piv_rx} 0 ${finger_vis_off}" rpy="0 ${pi} 0"/>
       <material name="link_mat"/>
     </visual>
-    <!-- 指片实测 X -23.4~-6.5  Y -4.0~1.0  Z 35.0~94.3 (mm) -->
-    <collision>
-      <geometry><box size="0.0169 0.005 0.0593"/></geometry>
-      <origin xyz="-0.01495 -0.0015 0.06465" rpy="0 0 0"/>
+    <collision>
+      <geometry><box size="${finger_half_w*2} 0.005 ${finger_len}"/></geometry>
+      <origin xyz="0 -0.0015 ${finger_len/2}" rpy="0 0 0"/>
     </collision>
     <inertial>
@@ -363,11 +371,11 @@
     </inertial>
   </link>
-  <joint name="finger_right_joint" type="prismatic">
+  <joint name="finger_right_joint" type="revolute">
     <parent link="gripper_base_link"/>
     <child link="finger_right_link"/>
-    <origin xyz="0 0 0" rpy="0 0 0"/>
-    <axis xyz="1 0 0"/>
-    <limit lower="-${finger_stroke}" upper="0" effort="12.0" velocity="0.04"/>
-    <dynamics damping="2.0" friction="0.5"/>
+    <origin xyz="${finger_piv_rx} 0 ${finger_piv_z}" rpy="0 0 0"/>
+    <axis xyz="0 1 0"/>
+    <limit lower="-${lim_finger}" upper="0" effort="12.0" velocity="1.5"/>
+    <dynamics damping="2.0" friction="0.4"/>
     <mimic joint="finger_left_joint" multiplier="-1" offset="0"/>
   </joint>

Commit message: feat(gripper): 补上张开时爪尖的回缩（等效四连杆），两指各加一级 mimic 滑座
用户补了一张合拢态带尺子的实拍：尺子 0 对准齿轮中心、沿爪身量到爪尖，
读数是 8.3~8.5cm，两爪尖相距约 0.7cm。三点与模型完全一致
（模型 85.1 / 7.8mm），说明「齿轮中心→爪尖」这个基准没问题。

于是「合拢 85 / 全开 70」这 15mm 的差就不是测量误差，而是机构本身：
爪尖张开时一边外摆一边朝齿轮方向回缩 —— 单铰转动做不出来（模型只到 82.5），
实机是四连杆，爪尖走耦合曲线。

- xacro：每根手指在转动关节之前串一级 prismatic（axis 沿爪轴 -Z，
  0~finger_pullback=13.5mm），用 <mimic> 线性跟随 finger_left_joint，
  multiplier = finger_pullback/lim_finger = 0.03277。
  置 finger_pullback=0 即退回纯单铰模型。
- preview.html：面板过滤掉 mimic+prismatic 的内部补偿关节（行数仍是 7），
  applyAll 原有的 prismatic 分支直接复用。
- README ×2：关节表补 carriage、机构说明补回缩来由、尺寸依据补
  「全开齿轮中心→爪尖 70mm（轴向投影）」、待校准项改写。

验证（页面内量网格顶点，强制 updateMatrixWorld）：
  合拢  爪距 7.8mm / 齿轮→爪尖 85.1（直距）85.0（轴向）
  全开  爪距 56.3mm / 齿轮→爪尖 75.4（直距）**69.9**（轴向）
轴向 69.9 对上实测 70；URDF 树校验：13 link / 12 joint，单根 world，无悬挂。

File: k3b_arm_urdf/k3b_arm.urdf (robot description, URDF)
Before this commit: robot k3b_arm, 11 links, 10 joints
Links:
- added link finger_left_carriage_link, mass 0.005
- added link finger_right_carriage_link, mass 0.005
Joints:
- added joint finger_left_carriage_joint: type prismatic, parent gripper_base_link, child finger_left_carriage_link, origin xyz=0 0 0 rpy=0 0 0, axis 0 0 -1, limit lower=0 upper=0.0135 effort=20.0 velocity=0.2, mimic joint=finger_left_joint multiplier=0.032766990291262135 offset=0
- added joint finger_right_carriage_joint: type prismatic, parent gripper_base_link, child finger_right_carriage_link, origin xyz=0 0 0 rpy=0 0 0, axis 0 0 -1, limit lower=0 upper=0.0135 effort=20.0 velocity=0.2, mimic joint=finger_left_joint multiplier=0.032766990291262135 offset=0
- joint finger_left_joint: parent gripper_base_link -> finger_left_carriage_link
- joint finger_right_joint: parent gripper_base_link -> finger_right_carriage_link

File: k3b_arm_urdf/k3b_arm.urdf.xacro (robot description, xacro)
@@ -48,4 +48,9 @@
   <!-- 指片转角限位：0 = 合拢（内距 7.5mm），0.400rad(22.9°) = 全开（内距 55mm） -->
   <xacro:property name="lim_finger" value="0.412"/>
+  <!-- 张开时爪尖的回缩量（m）。实机是四连杆，爪尖走的是耦合曲线：
+       合拢 85mm -> 全开 70mm，即张开过程爪尖同时向内收约 13.5mm。
+       单个转动关节做不出这一段，用「沿爪轴平移」等效补偿。
+       纯转动模型（不补偿）把这里置 0 即可。 -->
+  <xacro:property name="finger_pullback" value="0.0135"/>
   <!-- 指片转轴（取指片顶端中心），claw 系 -> link 系后 -->
   <xacro:property name="finger_piv_lx" value="0.00945"/>
@@ -347,6 +352,21 @@
     </inertial>
   </link>
+  <!-- 滑座：等效四连杆的「爪尖内收」，沿爪轴 -Z 平移，随指片转角线性跟随 -->
+  <link name="finger_left_carriage_link">
+    <inertial>
+      <mass value="0.005"/>
+      <inertia ixx="0.000001" ixy="0.0" ixz="0.0" iyy="0.000001" iyz="0.0" izz="0.000001"/>
+    </inertial>
+  </link>
+  <joint name="finger_left_carriage_joint" type="prismatic">
+    <parent link="gripper_base_link"/>
+    <child link="finger_left_carriage_link"/>
+    <origin xyz="0 0 0" rpy="0 0 0"/>
+    <axis xyz="0 0 -1"/>
+    <limit lower="0" upper="${finger_pullback}" effort="20.0" velocity="0.2"/>
+    <mimic joint="finger_left_joint" multiplier="${finger_pullback/lim_finger}" offset="0"/>
+  </joint>
   <joint name="finger_left_joint" type="revolute">
-    <parent link="gripper_base_link"/>
+    <parent link="finger_left_carriage_link"/>
     <child link="finger_left_link"/>
     <origin xyz="${finger_piv_lx} 0 ${finger_piv_z}" rpy="0 0 0"/>
@@ -371,6 +391,20 @@
     </inertial>
   </link>
+  <link name="finger_right_carriage_link">
+    <inertial>
+      <mass value="0.005"/>
+      <inertia ixx="0.000001" ixy="0.0" ixz="0.0" iyy="0.000001" iyz="0.0" izz="0.000001"/>
+    </inertial>
+  </link>
+  <joint name="finger_right_carriage_joint" type="prismatic">
+    <parent link="gripper_base_link"/>
+    <child link="finger_right_carriage_link"/>
+    <origin xyz="0 0 0" rpy="0 0 0"/>
+    <axis xyz="0 0 -1"/>
+    <limit lower="0" upper="${finger_pullback}" effort="20.0" velocity="0.2"/>
+    <mimic joint="finger_left_joint" multiplier="${finger_pullback/lim_finger}" offset="0"/>
+  </joint>
   <joint name="finger_right_joint" type="revolute">
-    <parent link="gripper_base_link"/>
+    <parent link="finger_right_carriage_link"/>
     <child link="finger_right_link"/>
     <origin xyz="${finger_piv_rx} 0 ${finger_piv_z}" rpy="0 0 0"/>
