Commit message: feat(gripper): 实机真四连杆 —— 21 分件按运动副拆成 7 块，销孔反解杆长与 mimic
先把 part_claw.stl 的 21 个连通分件按运动副重新归堆：
  claw_body(8,384) / claw_gear_left(4,396) / claw_gear_right(1,360)
  / claw_finger_left,right(14,796) / claw_bar_left,right(1,416)
面数之和 = 46,564 = 原文件，无遗漏。原来把连杆与齿轮臂都并进壳体的做法作废。

再用 STL 内部孔洞检测（flood fill 外部 + 内部连通域）读出所有销孔坐标，
按「孔位共点」定出拓扑：
  机身 ─G─ 齿轮臂 ─A─ 指片 ─B─ 平行连杆 ─R─ 机身
  rocker1 29.98 / coupler 21.01 / rocker2 29.96 / ground 22.34 mm
Grashof：21.01+29.98 = 50.99 < 52.30，最短杆是 coupler -> 双摇杆，齿轮臂只摆动。

新增 tools/claw_4bar.py（圆-圆交点法解四连杆 + 开合扫描）与
tools/emit_gripper.py（幂等写回 xacro），删除已被证伪的 solve_gripper.py。

URDF 变化：
- S1 改为驱动 finger_left_gear_joint（0~0.95993 rad），其余 5 个关节全为 mimic
- mimic_finger = -1.12343（相对齿轮臂）、mimic_bar = +0.94140
- 右指整条链 axis=(0 -1 0)，天然镜像；不再有 prismatic 滑座

结果：合拢 7.50mm / 84.30mm，全开 41.92mm / 67.96mm（实测 7.5 / 85、55 / 70）。
轴向吻合、开度差 13mm —— 该四连杆硬极限（齿轮 80°）也只有 47mm 内距，
判定实测 55mm 量的不是爪尖内角，已在文档中标为待复测项。

顺手：expand.py 把绝对路径写进注释头的问题修掉（改为仓库内相对路径，跨机器 diff 稳定）。

File: k3b_arm_urdf/k3b_arm.urdf (robot description, URDF)
Before this commit: robot k3b_arm, 13 links, 12 joints
Links:
- removed link finger_left_carriage_link
- removed link finger_right_carriage_link
- added link finger_left_bar_link, mass 0.015; collision box size=0.010 0.011 0.030; visual mesh filename=package://k3b_arm_urdf/meshes/claw_bar_left.stl
- added link finger_left_gear_link, mass 0.03; collision box size=0.028 0.006 0.050; visual mesh filename=package://k3b_arm_urdf/meshes/claw_gear_left.stl
- added link finger_right_bar_link, mass 0.015; collision box size=0.010 0.011 0.030; visual mesh filename=package://k3b_arm_urdf/meshes/claw_bar_right.stl
- added link finger_right_gear_link, mass 0.03; collision box size=0.028 0.006 0.050; visual mesh filename=package://k3b_arm_urdf/meshes/claw_gear_right.stl
- link finger_left_link: geometry collision box size=0.0169 0.005 0.0593; visual mesh filename=package://k3b_arm_urdf/meshes/claw_finger_left.stl
- link finger_right_link: geometry collision box size=0.0169 0.005 0.0593; visual mesh filename=package://k3b_arm_urdf/meshes/claw_finger_right.stl
- link gripper_base_link: mass 0.1 -> 0.12; geometry collision box size=0.060 0.024 0.050; visual mesh filename=package://k3b_arm_urdf/meshes/claw_body.stl
Joints:
- removed joint finger_left_carriage_joint
- removed joint finger_right_carriage_joint
- added joint finger_left_bar_joint: type revolute, parent gripper_base_link, child finger_left_bar_link, origin xyz=0.00505 0 0.0184 rpy=0 0 0, axis 0 1 0, limit lower=0 upper=0.903678102 effort=8.0 velocity=1.5, mimic joint=finger_left_gear_joint multiplier=0.9414 offset=0
- added joint finger_left_gear_joint: type revolute, parent gripper_base_link, child finger_left_gear_link, origin xyz=0.01345 0 -0.0023 rpy=0 0 0, axis 0 1 0, limit lower=0 upper=0.95993 effort=12.0 velocity=2.0
- added joint finger_right_bar_joint: type revolute, parent gripper_base_link, child finger_right_bar_link, origin xyz=-0.00505 0 0.0184 rpy=0 0 0, axis 0 -1 0, limit lower=0 upper=0.903678102 effort=8.0 velocity=1.5, mimic joint=finger_left_gear_joint multiplier=0.9414 offset=0
- added joint finger_right_gear_joint: type revolute, parent gripper_base_link, child finger_right_gear_link, origin xyz=-0.01345 0 -0.0023 rpy=0 0 0, axis 0 -1 0, limit lower=0 upper=0.95993 effort=12.0 velocity=2.0, mimic joint=finger_left_gear_joint multiplier=1 offset=0
- joint finger_left_joint: limit lower=0 upper=0.412 effort=12.0 velocity=1.5 -> lower=-1.0784141599 upper=0 effort=8.0 velocity=1.5; mimic (none) -> joint=finger_left_gear_joint multiplier=-1.12343 offset=0; origin xyz=0.00945 0 0.0227 rpy=0 0 0 -> xyz=0.00220 0 0.0299 rpy=0 0 0; parent finger_left_carriage_link -> finger_left_gear_link
- joint finger_right_joint: axis 0 1 0 -> 0 -1 0; limit lower=-0.412 upper=0 effort=12.0 velocity=1.5 -> lower=-1.0784141599 upper=0 effort=8.0 velocity=1.5; mimic joint=finger_left_joint multiplier=-1 offset=0 -> joint=finger_left_gear_joint multiplier=-1.12343 offset=0; origin xyz=-0.01495 0 0.0227 rpy=0 0 0 -> xyz=-0.00220 0 0.0299 rpy=0 0 0; parent finger_right_carriage_link -> finger_right_gear_link

File: k3b_arm_urdf/k3b_arm.urdf.xacro (robot description, xacro)
@@ -38,27 +38,39 @@
   <xacro:property name="lim_wpitch" value="2.2340"/>   <!-- S5  270°  ±128° -->
   <xacro:property name="joint_speed" value="1.5"/>
-  <!-- ===== 夹爪（实测定，见 tools/solve_gripper.py） =====
-       claw 网格自己的坐标系：爪尖 Z=-54.3、爪顶 Z=+54.3、厚 Y=+-11
-       齿轮中心 = 爪尖往 +Z 量 85mm  =>  claw Z=+30.7
-       腕滚转输出 -> 爪尖 110mm、爪长 108.6mm  =>  爪顶几乎贴住腕轴
-       claw 网格原点距 gripper_base = 54.3 - 28 + 1.4 = 27.7mm -->
-  <xacro:property name="claw_z" value="0.0277"/>
-  <xacro:property name="gear_x" value="-0.00275"/>   <!-- 齿轮中心，claw X=+2.75 镜像后 -->
-  <xacro:property name="gear_z" value="-0.0030"/>    <!-- 齿轮中心，爪顶下 23.6mm -->
-  <!-- 指片转角限位：0 = 合拢（内距 7.5mm），0.400rad(22.9°) = 全开（内距 55mm） -->
-  <xacro:property name="lim_finger" value="0.412"/>
-  <!-- 张开时爪尖的回缩量（m）。实机是四连杆，爪尖走的是耦合曲线：
-       合拢 85mm -> 全开 70mm，即张开过程爪尖同时向内收约 13.5mm。
-       单个转动关节做不出这一段，用「沿爪轴平移」等效补偿。
-       纯转动模型（不补偿）把这里置 0 即可。 -->
-  <xacro:property name="finger_pullback" value="0.0135"/>
-  <!-- 指片转轴（取指片顶端中心），claw 系 -> link 系后 -->
-  <xacro:property name="finger_piv_lx" value="0.00945"/>
-  <xacro:property name="finger_piv_rx" value="-0.01495"/>
-  <xacro:property name="finger_piv_z" value="0.0227"/>
-  <!-- 指片 visual 原点补偿：claw_z - 转轴 z（转轴在指片顶端，不在 claw 原点） -->
-  <xacro:property name="finger_vis_off" value="${claw_z - finger_piv_z}"/>
-  <xacro:property name="finger_half_w" value="0.00845"/>  <!-- 指片半宽（X） -->
-  <xacro:property name="finger_len" value="0.0593"/>      <!-- 指片长（Z） -->
+  <!-- ===== 夹爪：真四连杆（孔位反解，见 tools/claw_4bar.py） =====
+       part_claw.stl 的 21 个连通分件按「孔位共点」关系，确定是一条四连杆链：
+           机身 ──G── 齿轮臂 ──A── 指片 ──B── 平行连杆 ──R── 机身
+          (ground)  rocker1   coupler   rocker2        (ground)
+          杆长 30.0          21.0        30.0          22.3  mm
+       S1 输出轴带一只齿轮扇形板，与另一只扇形板啮合，两者转向相反 ——
+       所以左右两指严格镜像；右指全部 mimic 左指，轴取 (0 -1 0)。
+       本块所有坐标都在 gripper_base 系，对称面 = X=0、爪轴 = +Z
+       （claw 网格 Xc=2.75 / Zc=+27.7 映射到原点，见 claw_x / claw_z）。 -->
+  <xacro:property name="claw_x" value="0.00275"/>   <!-- claw 网格对称面 -->
+  <xacro:property name="claw_z" value="0.02770"/>   <!-- claw 网格 -> gripper_base -->
+  <!-- G 齿轮轴心 -->
+  <xacro:property name="gear_u" value="0.01345"/>
+  <xacro:property name="gear_z" value="-0.00230"/>
+  <xacro:property name="gear_v" value="0.03000"/>
+  <!-- R 平行连杆根部销 -->
+  <xacro:property name="bar_u"  value="0.00505"/>
+  <xacro:property name="bar_z"  value="0.01840"/>
+  <xacro:property name="bar_v"  value="0.00930"/>
+  <!-- A 指根销（相对齿轮轴） -->
+  <xacro:property name="pa_u"   value="0.00220"/>
+  <xacro:property name="pa_z"   value="0.02990"/>
+  <xacro:property name="pa_v"   value="0.00010"/>
+  <!-- S1：输出轴落在齿轮轴心上，机身向 +Y 外挂 -->
+  <xacro:property name="s1_x" value="-0.02348"/>
+  <xacro:property name="s1_y" value="0.012"/>
+  <!-- 行程：S1 850~1500μs -> 齿轮臂 0~55°。55° 时齿轮中心→爪尖 = 68.0mm（实测 70）；
+       机构硬极限在 80°（指间内距 47mm），先到的是舵机行程。 -->
+  <xacro:property name="lim_gear" value="0.95993"/>
+  <!-- 从动件 mimic 系数：按 55° 端点匹配（URDF mimic 只能线性，中段为近似） -->
+  <xacro:property name="mimic_finger" value="-1.12343"/>
+  <xacro:property name="mimic_bar"    value="0.94140"/>
+  <!-- 各杆碰撞盒（粗） -->
+  <xacro:property name="finger_half_w" value="0.00845"/>
+  <xacro:property name="finger_len" value="0.0593"/>
   <!-- ================= 网格 ================= -->
   <xacro:property name="mesh_dir" value="package://k3b_arm_urdf/meshes/"/>
@@ -294,27 +306,24 @@
     <dynamics damping="0.1" friction="0.05"/>
   </joint>
-  <!-- ================= 夹爪 ================= -->
-  <!-- 装配基准由实测定（见 tools/solve_gripper.py）：
-       齿轮中心 -> 爪尖 85mm，腕滚转输出 -> 爪尖 110mm，爪长 108.6mm
-       所以爪顶几乎就贴在腕滚转轴上，claw 网格原点距 gripper_base 27.7mm。 -->
+  <!-- ================= 夹爪机身（固定，含 S1） ================= -->
   <link name="gripper_base_link">
-    <!-- S1：输出轴接一只齿轮（= 齿轮中心），机身从爪体 +Y 面外挂 -->
+    <!-- S1：输出轴对准齿轮轴心，机身从爪体 +Y 面外挂 -->
     <visual>
       <geometry><mesh filename="${mesh_dir}s20f.stl"/></geometry>
-      <origin xyz="${gear_x} 0.013 ${gear_z}" rpy="${pi/2} 0 0"/>
+      <origin xyz="${s1_x} ${s1_y} ${gear_z}" rpy="${pi/2} 0 0"/>
       <material name="servo_mat"/>
     </visual>
-    <!-- 新款机械爪：壳体 + 平行连杆 + 齿轮组 -->
+    <!-- 机械爪壳体：背板 + 舵机支架 + 垫块（齿轮扇形板与连杆已拆成独立杆件） -->
     <visual>
       <geometry><mesh filename="${mesh_dir}claw_body.stl"/></geometry>
-      <origin xyz="0 0 ${claw_z}" rpy="0 ${pi} 0"/>
-      <material name="metal_mat"/>
-    </visual>
-    <collision>
-      <geometry><box size="0.060 0.022 0.078"/></geometry>
-      <origin xyz="0 0 0.0124" rpy="0 0 0"/>
-    </collision>
-    <inertial>
-      <mass value="0.1"/>
+      <origin xyz="${claw_x} 0 ${claw_z}" rpy="0 ${pi} 0"/>
+      <material name="metal_mat"/>
+    </visual>
+    <collision>
+      <geometry><box size="0.060 0.024 0.050"/></geometry>
+      <origin xyz="0 0 0.025" rpy="0 0 0"/>
+    </collision>
+    <inertial>
+      <mass value="0.12"/>
       <inertia ixx="0.0001" ixy="0.0" ixz="0.0" iyy="0.0001" iyz="0.0" izz="0.0001"/>
     </inertial>
@@ -325,5 +334,5 @@
     <origin xyz="0 0 0.028" rpy="0 0 0"/>
   </joint>
-  <!-- 末端工具坐标系（抓取参考点，落在爪尖） -->
+  <!-- 末端工具坐标系：两爪尖正中间 -->
   <link name="tool0"/>
   <joint name="tool0_joint" type="fixed">
@@ -332,18 +341,39 @@
     <origin xyz="0 0 0.082" rpy="0 0 0"/>
   </joint>
-  <!-- ================= J6 左指（S1 经齿轮驱动） ================= -->
-  <!-- 机构：S1 输出轴带一只齿轮，与指片根部的齿轮啮合；两齿轮转向相反，
-       所以两指反向等角摆开 —— 正好就是 mimic multiplier=-1。
-       指片绕自身顶端中心转动（取该点为转轴），0 = 合拢，0.400rad = 全开。 -->
+  <!-- ================= 左齿轮扇形板（S1 侧 / 啮合侧） ================= -->
+  <!-- 输入杆：S1 直接驱动。正向 = 张开（逆时针） -->
+  <link name="finger_left_gear_link">
+    <visual>
+      <geometry><mesh filename="${mesh_dir}claw_gear_left.stl"/></geometry>
+      <origin xyz="-0.01070 0 ${gear_v}" rpy="0 ${pi} 0"/>
+      <material name="metal_mat"/>
+    </visual>
+    <collision>
+      <geometry><box size="0.028 0.006 0.050"/></geometry>
+      <origin xyz="0 0 0.015" rpy="0 0 0"/>
+    </collision>
+    <inertial>
+      <mass value="0.03"/>
+      <inertia ixx="0.00001" ixy="0.0" ixz="0.0" iyy="0.00001" iyz="0.0" izz="0.00001"/>
+    </inertial>
+  </link>
+  <joint name="finger_left_gear_joint" type="revolute">
+    <parent link="gripper_base_link"/>
+    <child link="finger_left_gear_link"/>
+    <origin xyz="0.01345 0 ${gear_z}" rpy="0 0 0"/>
+    <axis xyz="0 1 0"/>
+    <limit lower="0" upper="${lim_gear}" effort="12.0" velocity="2.0"/>
+    <dynamics damping="0.5" friction="0.1"/>
+  </joint>
+  <!-- ================= 左指片（连杆 coupler） ================= -->
   <link name="finger_left_link">
     <visual>
-      <geometry><mesh filename="${mesh_dir}finger_left.stl"/></geometry>
-      <origin xyz="${-finger_piv_lx} 0 ${finger_vis_off}" rpy="0 ${pi} 0"/>
+      <geometry><mesh filename="${mesh_dir}claw_finger_left.stl"/></geometry>
+      <origin xyz="-0.01290 0 ${pa_v}" rpy="0 ${pi} 0"/>
       <material name="link_mat"/>
     </visual>
-    <!-- 转轴系下：X ±8.45、Y -4..1、Z 0..59.3 (mm) -->
     <collision>
       <geometry><box size="${finger_half_w*2} 0.005 ${finger_len}"/></geometry>
-      <origin xyz="0 -0.0015 ${finger_len/2}" rpy="0 0 0"/>
+      <origin xyz="-0.0035 -0.0015 0.0247" rpy="0 0 0"/>
     </collision>
     <inertial>
@@ -352,37 +382,74 @@
     </inertial>
   </link>
-  <!-- 滑座：等效四连杆的「爪尖内收」，沿爪轴 -Z 平移，随指片转角线性跟随 -->
-  <link name="finger_left_carriage_link">
-    <inertial>
-      <mass value="0.005"/>
-      <inertia ixx="0.000001" ixy="0.0" ixz="0.0" iyy="0.000001" iyz="0.0" izz="0.000001"/>
-    </inertial>
-  </link>
-  <joint name="finger_left_carriage_joint" type="prismatic">
+  <joint name="finger_left_joint" type="revolute">
+    <parent link="finger_left_gear_link"/>
+    <child link="finger_left_link"/>
+    <origin xyz="0.00220 0 ${pa_z}" rpy="0 0 0"/>
+    <axis xyz="0 1 0"/>
+    <limit lower="${mimic_finger*lim_gear}" upper="0" effort="8.0" velocity="1.5"/>
+    <mimic joint="finger_left_gear_joint" multiplier="${mimic_finger}" offset="0"/>
+    <dynamics damping="1.0" friction="0.2"/>
+  </joint>
+  <!-- ================= 左平行连杆（rocker2） ================= -->
+  <link name="finger_left_bar_link">
+    <visual>
+      <geometry><mesh filename="${mesh_dir}claw_bar_left.stl"/></geometry>
+      <origin xyz="-0.00230 0 ${bar_v}" rpy="0 ${pi} 0"/>
+      <material name="metal_mat"/>
+    </visual>
+    <collision>
+      <geometry><box size="0.010 0.011 0.030"/></geometry>
+      <origin xyz="-0.0026 0 -0.0052" rpy="0 0 0"/>
+    </collision>
+    <inertial>
+      <mass value="0.015"/>
+      <inertia ixx="0.000005" ixy="0.0" ixz="0.0" iyy="0.000005" iyz="0.0" izz="0.000005"/>
+    </inertial>
+  </link>
+  <joint name="finger_left_bar_joint" type="revolute">
     <parent link="gripper_base_link"/>
-    <child link="finger_left_carriage_link"/>
-    <origin xyz="0 0 0" rpy="0 0 0"/>
-    <axis xyz="0 0 -1"/>
-    <limit lower="0" upper="${finger_pullback}" effort="20.0" velocity="0.2"/>
-    <mimic joint="finger_left_joint" multiplier="${finger_pullback/lim_finger}" offset="0"/>
-  </joint>
-  <joint name="finger_left_joint" type="revolute">
-    <parent link="finger_left_carriage_link"/>
-    <child link="finger_left_link"/>
-    <origin xyz="${finger_piv_lx} 0 ${finger_piv_z}" rpy="0 0 0"/>
+    <child link="finger_left_bar_link"/>
+    <origin xyz="0.00505 0 ${bar_z}" rpy="0 0 0"/>
     <axis xyz="0 1 0"/>
-    <limit lower="0" upper="${lim_finger}" effort="12.0" velocity="1.5"/>
-    <dynamics damping="2.0" friction="0.4"/>
-  </joint>
-  <!-- ================= J6 右指（齿轮啮合，反向跟随） ================= -->
+    <limit lower="0" upper="${mimic_bar*lim_gear}" effort="8.0" velocity="1.5"/>
+    <mimic joint="finger_left_gear_joint" multiplier="${mimic_bar}" offset="0"/>
+    <dynamics damping="1.0" friction="0.2"/>
+  </joint>
+  <!-- ================= 右齿轮扇形板（S1 侧 / 啮合侧） ================= -->
+  <!-- 与左齿轮啮合，转向相反 -> axis 取 -Y，mimic 系数 +1 即为镜像 -->
+  <link name="finger_right_gear_link">
+    <visual>
+      <geometry><mesh filename="${mesh_dir}claw_gear_right.stl"/></geometry>
+      <origin xyz="0.01620 0 ${gear_v}" rpy="0 ${pi} 0"/>
+      <material name="metal_mat"/>
+    </visual>
+    <collision>
+      <geometry><box size="0.028 0.006 0.050"/></geometry>
+      <origin xyz="0 0 0.015" rpy="0 0 0"/>
+    </collision>
+    <inertial>
+      <mass value="0.03"/>
+      <inertia ixx="0.00001" ixy="0.0" ixz="0.0" iyy="0.00001" iyz="0.0" izz="0.00001"/>
+    </inertial>
+  </link>
+  <joint name="finger_right_gear_joint" type="revolute">
+    <parent link="gripper_base_link"/>
+    <child link="finger_right_gear_link"/>
+    <origin xyz="-0.01345 0 ${gear_z}" rpy="0 0 0"/>
+    <axis xyz="0 -1 0"/>
+    <limit lower="0" upper="${lim_gear}" effort="12.0" velocity="2.0"/>
+    <mimic joint="finger_left_gear_joint" multiplier="1" offset="0"/>
+    <dynamics damping="0.5" friction="0.1"/>
+  </joint>
+  <!-- ================= 右指片（连杆 coupler） ================= -->
   <link name="finger_right_link">
     <visual>
-      <geometry><mesh filename="${mesh_dir}finger_right.stl"/></geometry>
-      <origin xyz="${-finger_piv_rx} 0 ${finger_vis_off}" rpy="0 ${pi} 0"/>
+      <geometry><mesh filename="${mesh_dir}claw_finger_right.stl"/></geometry>
+      <origin xyz="0.01840 0 ${pa_v}" rpy="0 ${pi} 0"/>
       <material name="link_mat"/>
     </visual>
     <collision>
       <geometry><box size="${finger_half_w*2} 0.005 ${finger_len}"/></geometry>
-      <origin xyz="0 -0.0015 ${finger_len/2}" rpy="0 0 0"/>
+      <origin xyz="-0.0035 -0.0015 0.0247" rpy="0 0 0"/>
     </collision>
     <inertial>
@@ -391,26 +458,37 @@
     </inertial>
   </link>
-  <link name="finger_right_carriage_link">
-    <inertial>
-      <mass value="0.005"/>
-      <inertia ixx="0.000001" ixy="0.0" ixz="0.0" iyy="0.000001" iyz="0.0" izz="0.000001"/>
-    </inertial>
-  </link>
-  <joint name="finger_right_carriage_joint" type="prismatic">
+  <joint name="finger_right_joint" type="revolute">
+    <parent link="finger_right_gear_link"/>
+    <child link="finger_right_link"/>
+    <origin xyz="-0.00220 0 ${pa_z}" rpy="0 0 0"/>
+    <axis xyz="0 -1 0"/>
+    <limit lower="${mimic_finger*lim_gear}" upper="0" effort="8.0" velocity="1.5"/>
+    <mimic joint="finger_left_gear_joint" multiplier="${mimic_finger}" offset="0"/>
+    <dynamics damping="1.0" friction="0.2"/>
+  </joint>
+  <!-- ================= 右平行连杆（rocker2） ================= -->
+  <link name="finger_right_bar_link">
+    <visual>
+      <geometry><mesh filename="${mesh_dir}claw_bar_right.stl"/></geometry>
+      <origin xyz="0.00780 0 ${bar_v}" rpy="0 ${pi} 0"/>
+      <material name="metal_mat"/>
+    </visual>
+    <collision>
+      <geometry><box size="0.010 0.011 0.030"/></geometry>
+      <origin xyz="-0.0026 0 -0.0052" rpy="0 0 0"/>
+    </collision>
+    <inertial>
+      <mass value="0.015"/>
+      <inertia ixx="0.000005" ixy="0.0" ixz="0.0" iyy="0.000005" iyz="0.0" izz="0.000005"/>
+    </inertial>
+  </link>
+  <joint name="finger_right_bar_joint" type="revolute">
     <parent link="gripper_base_link"/>
-    <child link="finger_right_carriage_link"/>
-    <origin xyz="0 0 0" rpy="0 0 0"/>
-    <axis xyz="0 0 -1"/>
-    <limit lower="0" upper="${finger_pullback}" effort="20.0" velocity="0.2"/>
-    <mimic joint="finger_left_joint" multiplier="${finger_pullback/lim_finger}" offset="0"/>
-  </joint>
-  <joint name="finger_right_joint" type="revolute">
-    <parent link="finger_right_carriage_link"/>
-    <child link="finger_right_link"/>
-    <origin xyz="${finger_piv_rx} 0 ${finger_piv_z}" rpy="0 0 0"/>
-    <axis xyz="0 1 0"/>
-    <limit lower="-${lim_finger}" upper="0" effort="12.0" velocity="1.5"/>
-    <dynamics damping="2.0" friction="0.4"/>
-    <mimic joint="finger_left_joint" multiplier="-1" offset="0"/>
+    <child link="finger_right_bar_link"/>
+    <origin xyz="-0.00505 0 ${bar_z}" rpy="0 0 0"/>
+    <axis xyz="0 -1 0"/>
+    <limit lower="0" upper="${mimic_bar*lim_gear}" effort="8.0" velocity="1.5"/>
+    <mimic joint="finger_left_gear_joint" multiplier="${mimic_bar}" offset="0"/>
+    <dynamics damping="1.0" friction="0.2"/>
   </joint>
   <!-- ================= 世界坐标系 ================= -->

Commit message: fix(gripper): 用实拍钢尺照片反标定行程，lim_gear 55°→80°（机构锁死角）
用户补了一张「全开 + 钢尺」照片，尺 0 放在上爪齿尖。做了定量标定：

1. 尺子 mm 刻度列连续刻度线的 y 中位间距 = 12.5 px/mm（上段 12.65 / 下段 12.45，
   分段线性换算补透视）；
2. 用画面里 M3 内六角圆柱头螺钉（标准头径 5.5mm）交叉验证 → 11.8 px/mm，
   两种基准差 5%，标定可信；
3. 上爪齿尖 y=372、下爪齿尖 y=997 → 4.1mm / 53.8mm → **全开内距 ≈ 49.7mm**
   （按螺钉基准则 ≈53mm）。

之前拿「齿轮中心→爪尖 70mm」反推出 S1 只走 55°，导致全开内距只有 41.9mm —— 偏小。
现在改成走满机构行程：

  lim_gear     0.95993 -> 1.39626 rad (55° -> 80°)
  mimic_finger -1.12343 -> -1.10533
  mimic_bar    +0.94140 -> +0.96141

合拢 7.50 / 84.30mm（不变）；全开 41.92 / 67.96 → **47.07 / 55.09mm**。

仍差 3~6mm：47.07 是这套四连杆的数学上限（θ=79° 内距最大，再转回缩）。
差额可能来自销孔配合间隙或齿扇背隙。已在 README 把「lim_gear 实机标定」列为校准第一项，
给出「打满 S1 → 量爪距 → 回查扫描表定角 → 改 TH_MAX 重跑 emit_gripper」的闭环。

顺带：claw_4bar 的报告修正了扫描方向（原来扫负角，误报「未达到」），
并补上最大内距统计与 mimic 系数打印；emit_gripper 的 TH_MAX 改为从 claw_4bar 导入，
两边不再可能不同步。

File: k3b_arm_urdf/k3b_arm.urdf (robot description, URDF)
Before this commit: robot k3b_arm, 15 links, 14 joints
Joints:
- joint finger_left_bar_joint: limit lower=0 upper=0.903678102 effort=8.0 velocity=1.5 -> lower=0 upper=1.3423783266 effort=8.0 velocity=1.5; mimic joint=finger_left_gear_joint multiplier=0.9414 offset=0 -> joint=finger_left_gear_joint multiplier=0.96141 offset=0
- joint finger_left_gear_joint: limit lower=0 upper=0.95993 effort=12.0 velocity=2.0 -> lower=0 upper=1.39626 effort=12.0 velocity=2.0
- joint finger_left_joint: limit lower=-1.0784141599 upper=0 effort=8.0 velocity=1.5 -> lower=-1.5433280658 upper=0 effort=8.0 velocity=1.5; mimic joint=finger_left_gear_joint multiplier=-1.12343 offset=0 -> joint=finger_left_gear_joint multiplier=-1.10533 offset=0
- joint finger_right_bar_joint: limit lower=0 upper=0.903678102 effort=8.0 velocity=1.5 -> lower=0 upper=1.3423783266 effort=8.0 velocity=1.5; mimic joint=finger_left_gear_joint multiplier=0.9414 offset=0 -> joint=finger_left_gear_joint multiplier=0.96141 offset=0
- joint finger_right_gear_joint: limit lower=0 upper=0.95993 effort=12.0 velocity=2.0 -> lower=0 upper=1.39626 effort=12.0 velocity=2.0
- joint finger_right_joint: limit lower=-1.0784141599 upper=0 effort=8.0 velocity=1.5 -> lower=-1.5433280658 upper=0 effort=8.0 velocity=1.5; mimic joint=finger_left_gear_joint multiplier=-1.12343 offset=0 -> joint=finger_left_gear_joint multiplier=-1.10533 offset=0

File: k3b_arm_urdf/k3b_arm.urdf.xacro (robot description, xacro)
@@ -4,5 +4,5 @@
   =============================================================
   执行器实测映射（2026-10-25）
-  S1  180° 位置   脉宽 850~1500   上电 850    → finger_left      行程 0~10mm
+  S1  180° 位置   脉宽 850~1500   上电 850    → finger_left_gear 0~80°（内距 7.5→47.1mm）
   S2  180° 位置   脉宽 500~2500   上电 1500   → base_yaw         限位 ±90°
   S3  270° 位置   脉宽 500~2000   上电 2000   → shoulder_pitch   限位 ±101°
@@ -11,5 +11,5 @@
   速度 360° 连续   无位置反馈      —          → wrist_roll       无限位(continuous)
   · S1~S4 为 WHEELTEC S20F，S5 为 PM15S（暂以 S20F 270° 代替，待实测修正）
-  · finger_right 用 mimic 跟随 finger_left，不单独接舵机
+  · 夹爪是真四连杆，只有 finger_left_gear 接 S1，其余 5 个关节全 mimic（见 tools/claw_4bar.py）
   · wrist_roll 是速度舵机、无位置反馈，MoveIt 逆解时需 disable
   机械件按实拍装配（套件为黑色阳极氧化支架 + 银色铝管 + 铝制平行连杆爪）：
@@ -64,10 +64,10 @@
   <xacro:property name="s1_x" value="-0.02348"/>
   <xacro:property name="s1_y" value="0.012"/>
-  <!-- 行程：S1 850~1500μs -> 齿轮臂 0~55°。55° 时齿轮中心→爪尖 = 68.0mm（实测 70）；
-       机构硬极限在 80°（指间内距 47mm），先到的是舵机行程。 -->
-  <xacro:property name="lim_gear" value="0.95993"/>
+  <!-- 行程：齿轮臂 0~80°。80° 是机构锁死角（内距最大 47.1mm，再大就回缩），
+       所以 URDF 允许走满全行程，S1 的实际脉宽子区间由实机标定后再收窄。 -->
+  <xacro:property name="lim_gear" value="1.39626"/>
   <!-- 从动件 mimic 系数：按 55° 端点匹配（URDF mimic 只能线性，中段为近似） -->
-  <xacro:property name="mimic_finger" value="-1.12343"/>
-  <xacro:property name="mimic_bar"    value="0.94140"/>
+  <xacro:property name="mimic_finger" value="-1.10533"/>
+  <xacro:property name="mimic_bar"    value="0.96141"/>
   <!-- 各杆碰撞盒（粗） -->
   <xacro:property name="finger_half_w" value="0.00845"/>
